File: IoT_2015/IoT_2015-1.sch (EAGLE design)
At the start: 28 parts, among them Y1 ABLS-16.000MHZ-B4-T

Commit message: Stop masks are corrected
All DRC errors are corrected. Specially the stop masks have been
corrected in the footprints of interest.
Parts:
- JTAG, P67VDD: device con-lstb:MA03-1 -> custom-con-lstb:MA03-1
Changed lines of the file:
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@@
 <?xml version="1.0" encoding="utf-8"?>
 <!DOCTYPE eagle SYSTEM "eagle.dtd">
-<eagle version="7.3.0">
+<eagle version="7.2.0">
 <drawing>
 <settings>
@@
 <part name="FRAME1" library="frames" deviceset="A3L-LOC" device=""/>
 <part name="GND13" library="supply1" deviceset="GND" device=""/>
-<part name="JTAG" library="con-lstb" deviceset="MA03-1" device=""/>
+<part name="JTAG" library="custom-con-lstb" deviceset="MA03-1" device=""/>
 <part name="ANTENNA" library="Pulse" deviceset="W3008" device=""/>
 <part name="SUPPLY6" library="supply2" deviceset="VDD" device=""/>
@@
 <part name="SUPPLY5" library="supply2" deviceset="VDD" device=""/>
 <part name="BATTERY" library="BAT-HLD-001" deviceset="BAT-HLD-001" device=""/>
-<part name="P67VDD" library="con-lstb" deviceset="MA03-1" device=""/>
+<part name="P67VDD" library="custom-con-lstb" deviceset="MA03-1" device=""/>
 <part name="GND16" library="supply1" deviceset="GND" device=""/>
 <part name="SUPPLY9" library="supply2" deviceset="VDD" device=""/>
